File: LightBoard-Gift/HardWare/LightBoard-Gift.kicad_sch (KiCad schematic)
At the start: 11 parts

Commit message: Work done so amazing
Parts:
- added SW1: SW_Push, Button_Switch_SMD:SW_Push_1P1T_NO_CK_KMR2, symbol Switch:SW_Push
Connections:
- net GND: now also SW1.2
- net at A1.29 (GPIO22): now also SW1.1
Changed lines of the file:
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@@
 	(generator_version "9.0")
 	(paper "A4")
+	(wire
+		(pts
+			(xy 175.26 44.45) (xy 177.8 44.45)
+		)
+		(stroke
+			(width 0)
+			(type default)
+		)
+	)
+	(wire
+		(pts
+			(xy 161.29 44.45) (xy 165.1 44.45)
+		)
+		(stroke
+			(width 0)
+			(type default)
+		)
+	)
 	(global_label "RED0"
 		(shape input)
@@
 				(justify right)
 				(hide yes)
+			)
+		)
+	)
+	(symbol
+		(lib_id "power:GND")
+		(at 177.8 44.45 90)
+		(unit 1)
+		(exclude_from_sim no)
+		(in_bom yes)
+		(on_board yes)
+		(dnp no)
+		(fields_autoplaced yes)
+		(property "Reference" "#PWR012"
+			(at 184.15 44.45 0)
+			(effects
+				(font
+					(size 1.27 1.27)
+				)
+				(hide yes)
+			)
+		)
+		(property "Value" "GND"
+			(at 181.61 44.4499 90)
+			(effects
+				(font
+					(size 1.27 1.27)
+				)
+				(justify right)
+			)
+		)
+		(property "Footprint" ""
+			(at 177.8 44.45 0)
+			(effects
+				(font
+					(size 1.27 1.27)
+				)
+				(hide yes)
+			)
+		)
+		(property "Datasheet" ""
+			(at 177.8 44.45 0)
+			(effects
+				(font
+					(size 1.27 1.27)
+				)
+				(hide yes)
+			)
+		)
+		(property "Description" "Power symbol creates a global label with name \"GND\" , ground"
+			(at 177.8 44.45 0)
+			(effects
+				(font
+					(size 1.27 1.27)
+				)
+				(hide yes)
+			)
+		)
+		(pin "1"
+		)
+		(instances
+			(project "LightBoard-Gift"
+				(path "/ee4ea1cd-56bb-4e48-b71d-bdae100177cd"
+					(reference "#PWR012")
+					(unit 1)
+				)
 			)
 		)
@@
 					(unit 1)
 				)
+			)
+		)
+	)
+	(symbol
+		(lib_id "Switch:SW_Push")
+		(at 170.18 44.45 0)
+		(unit 1)
+		(exclude_from_sim no)
+		(in_bom yes)
+		(on_board yes)
+		(dnp no)
+		(fields_autoplaced yes)
+		(property "Reference" "SW1"
+			(at 170.18 36.83 0)
+			(effects
+				(font
+					(size 1.27 1.27)
+				)
+			)
+		)
+		(property "Value" "SW_Push"
+			(at 170.18 39.37 0)
+			(effects
+				(font
+					(size 1.27 1.27)
+				)
+			)
+		)
+		(property "Footprint" "Button_Switch_SMD:SW_Push_1P1T_NO_CK_KMR2"
+			(at 170.18 39.37 0)
+			(effects
+				(font
+					(size 1.27 1.27)
+				)
+				(hide yes)
+			)
+		)
+		(property "Datasheet" "~"
+			(at 170.18 39.37 0)
+			(effects
+				(font
+					(size 1.27 1.27)
+				)
+				(hide yes)
+			)
+		)
+		(property "Description" "Push button switch, generic, two pins"
+			(at 170.18 44.45 0)
+			(effects
+				(font
+					(size 1.27 1.27)
+				)
+				(hide yes)
+			)
+		)
+		(pin "2"
+		)
+		(pin "1"
+		)
+		(instances
+			(project ""
+				(path "/ee4ea1cd-56bb-4e48-b71d-bdae100177cd"
+					(reference "SW1")
+					(unit 1)
+				)

Commit message: Silly additions
Parts:
- SW1: footprint Button_Switch_SMD:SW_Push_1P1T_NO_CK_KMR2 -> Button_Switch_THT:SW_PUSH_6mm_H4.3mm
Changed lines of the file:
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@@
 			)
 		)
-		(property "Footprint" "Button_Switch_SMD:SW_Push_1P1T_NO_CK_KMR2"
+		(property "Footprint" "Button_Switch_THT:SW_PUSH_6mm_H4.3mm"
 			(at 170.18 39.37 0)
 			(effects

Commit message: Lowkey?
Forgot to save the files before pushing the last commit
Parts:
- added H1, H2, H3, H4: MountingHole, MountingHole:MountingHole_2.2mm_M2, symbol Mechanical:MountingHole
- added R0, R1, R2, R4, R5, R6, R7, R8, R9: 560Ohm, Resistor_SMD:R_2512_6332Metric, symbol Device:R_Small
- added R3: R_Small, Resistor_SMD:R_2512_6332Metric, symbol Device:R_Small
- added SW2: SWITCH, Button_Switch_THT:SW_Slide_SPDT_Straight_CK_OS102011MS2Q, symbol Switch:SW_Push
- SW1: value SW_Push -> MODE_SELECT
Connections:
- net GND: now also SW2.1
- net RED0: now also A1.27 (GPIO21), R0.2; no longer A1.1 (GPIO0), D0.1 (RA)
- net RED1: now also A1.26 (GPIO20), R1.2; no longer A1.2 (GPIO1), D1.1 (RA)
- net RED2: now also A1.25 (GPIO19), R2.2; no longer A1.4 (GPIO2), D2.1 (RA)
- net RED3: now also A1.24 (GPIO18), R3.2; no longer A1.5 (GPIO3), D3.1 (RA)
- net RED4: now also A1.22 (GPIO17), R4.2; no longer A1.6 (GPIO4), D4.1 (RA)
- net RED5: now also A1.21 (GPIO16), R5.2; no longer A1.7 (GPIO5), D5.1 (RA)
- net RED6: now also A1.29 (GPIO22), R6.2; no longer A1.9 (GPIO6), D6.1 (RA)
- net RED7: now also A1.20 (GPIO15), R7.2; no longer A1.10 (GPIO7), D7.1 (RA)
- net RED8: now also A1.19 (GPIO14), R9.2; no longer A1.11 (GPIO8), D8.1 (RA)
- net RED9: now also A1.17 (GPIO13), R8.2; no longer A1.12 (GPIO9), D9.1 (RA)
- net at SW1.1: now also A1.1 (GPIO0); no longer A1.29 (GPIO22)
- new net: A1.6 (GPIO4), SW2.2
- new net: D3.1 (RA), R3.1
- new net: D4.1 (RA), R4.1
- new net: D5.1 (RA), R5.1
- new net: D2.1 (RA), R2.1
- new net: D8.1 (RA), R9.1
- new net: D1.1 (RA), R1.1
- new net: D0.1 (RA), R0.1
- new net: D7.1 (RA), R7.1
- new net: D9.1 (RA), R8.1
- new net: D6.1 (RA), R6.1
Other:
- moved on the sheet: D8, D9, SW1
