File: Lightboard-Gift-REMASTERED/Lightboard-Gift-REMASTERED.kicad_sch (KiCad schematic)
At the start: 20 parts, among them J1 USB_C_Receptacle_PowerOnly_6P, SW1 SW_Push, SW2 SW_SPST

Commit message: Work Hard Play Harder
Parts:
- added R10, R11, R12, R3, R4, R5, R6, R7, R8, R9: R_Small, Resistor_SMD:R_1812_4532Metric_Pad1.30x3.40mm_HandSolder, symbol Device:R_Small
Connections:
- net GND: now also A1.13 (GND), A1.18 (GND), A1.23 (GND), A1.28 (GND), A1.3 (GND), A1.33 (AGND), A1.38 (GND), A1.8 (GND), SW1.2; no longer SW1.1
- net RED0: now also A1.2 (GPIO1), R3.2; no longer A1.29 (GPIO22), D1.1 (RA)
- net RED1: now also A1.4 (GPIO2), R4.2; no longer A1.27 (GPIO21), D2.1 (RA)
- net RED2: now also A1.6 (GPIO4), R5.2; no longer A1.26 (GPIO20), D3.1 (RA)
- net RED3: now also A1.7 (GPIO5), R6.2; no longer A1.25 (GPIO19), D4.1 (RA)
- net RED4: now also A1.9 (GPIO6), R7.2; no longer A1.24 (GPIO18), D5.1 (RA)
- net RED5: now also A1.12 (GPIO9), R8.2; no longer A1.22 (GPIO17), D6.1 (RA)
- net RED6: now also A1.11 (GPIO8), R9.2; no longer A1.21 (GPIO16), D7.1 (RA)
- net RED7: now also A1.10 (GPIO7), R10.2; no longer A1.4 (GPIO2), D8.1 (RA)
- net RED8: now also A1.5 (GPIO3), R11.2; no longer A1.2 (GPIO1), D9.1 (RA)
- net RED9: now also R12.2; no longer D10.1 (RA)
- net at A1.20 (GPIO15): no longer SW1.2
- new net: D4.1 (RA), R6.1
- new net: D10.1 (RA), R12.1
- new net: D7.1 (RA), R9.1
- new net: D3.1 (RA), R5.1
- new net: D5.1 (RA), R7.1
- new net: D6.1 (RA), R8.1
- new net: D9.1 (RA), R11.1
- new net: D1.1 (RA), R3.1
- new net: A1.29 (GPIO22), SW1.1
- new net: D2.1 (RA), R4.1
- new net: D8.1 (RA), R10.1
Other:
- moved on the sheet: SW1
