File: 5gModem/5gModem/5gModem.kicad_pcb (KiCad board)
At the start: 2 copper layers, 69.4 x 57.2 mm, 8 parts, among them J1 USB_C_Receptacle_PowerOnly_6P, J2 USB_C_Receptacle_USB2.0_14P

Commit message: Worked a little
I think its far from done but I'm proud of what I have
Parts:
- removed R1, R2: 5k1, Resistor_SMD:R_1210_3225Metric_Pad1.30x2.65mm_HandSolder
Connections:
- J1 pad A5: Net-(J1-CC1) -> /CC1
- J1 pad B5: Net-(J1-CC2) -> /CC2
Routing:
- net /CC2: track 0.00 -> 45.1 mm
- net /CC1: track 0.00 -> 43.0 mm
- net GND: track 112.3 -> 136.4 mm, vias 63 -> 70
- net Net-(J1-CC2): track 5.15 -> 0.00 mm
- net Net-(J1-CC1): track 3.89 -> 0.00 mm
Other:
- outline, holes or cut-outs redrawn
- board text added: "DATA"
- board text added: "POWER"
