File: PiKeyboard/hardware/hardware.kicad_pcb (KiCad board)
At the start: 2 copper layers, 370 x 155 mm, 156 parts, among them J2 USB_C_Receptacle_PowerOnly_6P, J22 690-019-298-412, SW1 SW_Push, SW10 SW_Push, SW11 SW_Push, SW12 SW_Push, SW13 SW_Push, SW14 SW_Push, SW15 SW_Push, SW16 SW_Push, SW17 SW_Push, SW18 SW_Push, SW19 SW_Push, SW2 SW_Push, SW20 SW_Push, SW21 SW_Push, SW22 SW_Push, SW23 SW_Push, SW24 SW_Push, SW25 SW_Push, SW26 SW_Push, SW27 SW_Push, SW28 SW_Push, SW29 SW_Push, SW3 SW_Push, SW30 SW_Push, SW31 SW_Push, SW32 SW_Push, SW33 SW_Push, SW34 SW_Push, SW35 SW_Push, SW36 SW_Push, SW37 SW_Push, SW38 SW_Push, SW39 SW_Push, SW4 SW_Push, SW40 SW_Push, SW41 SW_Push, SW42 SW_Push, SW43 SW_Push, SW44 SW_Push, SW45 SW_Push, SW46 SW_Push, SW47 SW_Push, SW48 SW_Push, SW49 SW_Push, SW5 SW_Push, SW50 SW_Push, SW51 SW_Push, SW52 SW_Push, SW53 SW_Push, SW54 SW_Push, SW55 SW_Push, SW56 SW_Push, SW57 SW_Push, SW58 SW_Push, SW59 SW_Push, SW6 SW_Push, SW60 SW_Push, SW61 SW_Push, SW62 SW_Push, SW63 SW_Push, SW64 SW_Push, SW65 SW_Push, SW66 SW_Push, SW67 SW_Push, SW68 SW_Push, SW69 SW_Push, SW7 SW_Push, SW70 SW_Push, SW71 SW_Push, SW72 SW_Push, SW73 SW_Push, SW74 SW_Push, SW8 SW_Push, SW9 SW_Push, U12 RT9742SNGV

Commit message: yes
Parts:
- added C2: C_Small, Capacitor_SMD:C_0805_2012Metric_Pad1.18x1.45mm_HandSolder, B.Cu at (400.0, 217.2)
- J22: moved to B.Cu
- moved A1 95.4 mm to (366.4, 131.2), turned to 0 degrees
- moved Module1 83.1 mm to (394.7, 231.1)
- moved C1 23.1 mm to (380.3, 154.3)
- turned J22 to 0 degrees
Connections:
- A1 pad 1: C15 -> C5
- A1 pad 10: unconnected-(A1-GPIO7-Pad10) -> R5
- A1 pad 11: unconnected-(A1-GPIO8-Pad11) -> C11
- A1 pad 12: unconnected-(A1-GPIO9-Pad12) -> R4
- A1 pad 14: unconnected-(A1-GPIO10-Pad14) -> C12
- A1 pad 15: unconnected-(A1-GPIO11-Pad15) -> R3
- A1 pad 16: unconnected-(A1-GPIO12-Pad16) -> C13
- A1 pad 17: unconnected-(A1-GPIO13-Pad17) -> R2
- A1 pad 19: unconnected-(A1-GPIO14-Pad19) -> C14
- A1 pad 2: C14 -> C6
- A1 pad 20: unconnected-(A1-GPIO15-Pad20) -> R1
- A1 pad 4: R1 -> C7
- A1 pad 5: R2 -> C8
- A1 pad 6: C13 -> C9
- A1 pad 7: C12 -> R6
- A1 pad 9: C11 -> C10
- D50 pad 2: Net-(D50-A) -> Net-(D49-A)
- J22 pad 13: /HDMI0_CEC -> unconnected-(J22-CEC-Pad13)
- SW10 pad 1: C12 -> C11
- SW11 pad 1: C13 -> C12
- SW12 pad 1: C14 -> C13
- SW13 pad 1: C15 -> C14
- SW27 pad 1: C15 -> C14
- SW41 pad 1: C15 -> C14
- SW43 pad 1: C3 -> C2
- SW44 pad 1: C4 -> C3
- SW45 pad 1: C5 -> C4
- SW46 pad 1: C6 -> C5
- SW47 pad 1: C7 -> C6
- SW48 pad 1: C8 -> C7
- SW49 pad 1: C9 -> C8
- SW49 pad 2: Net-(D49-A) -> unconnected-(SW49-Pad2)
- SW50 pad 1: C10 -> C9
- SW50 pad 2: Net-(D50-A) -> Net-(D49-A)
- SW51 pad 1: C11 -> C10
- SW52 pad 1: C12 -> C11
- SW53 pad 1: C13 -> C12
- SW54 pad 1: C15 -> C14
- SW56 pad 1: C3 -> C2
- SW57 pad 1: C4 -> C3
- SW58 pad 1: C5 -> C4
- SW59 pad 1: C6 -> C5
- SW6 pad 1: C8 -> C7
- SW60 pad 1: C7 -> C6
- SW61 pad 1: C8 -> C7
- SW62 pad 1: C9 -> C8
- SW63 pad 1: C10 -> C9
- SW64 pad 1: C11 -> C10
- SW65 pad 1: C12 -> C11
- SW66 pad 1: C15 -> C14
- SW7 pad 1: C9 -> C8
- SW70 pad 1: C7 -> C6
- SW71 pad 1: C12 -> C10
- SW72 pad 1: C13 -> C11
- SW73 pad 1: C14 -> C13
- SW74 pad 1: C15 -> C14
- SW8 pad 1: C10 -> C9
- SW9 pad 1: C11 -> C10
Routing:
- net C5: track 98.6 -> 386.3 mm, vias 0 -> 1
- net C6: track 97.8 -> 361.5 mm, vias 0 -> 1
- net C7: track 91.0 -> 339.3 mm, vias 0 -> 1
- net C8: track 101.5 -> 320.8 mm, vias 0 -> 1
- net C9: track 102.5 -> 302.6 mm, vias 0 -> 1
- net C10: track 102.5 -> 281.0 mm, vias 0 -> 1
- net /HDMI0_HOTPLUG: track 0.00 -> 166.7 mm
- net C15: track 144.1 -> 0.00 mm, vias 1 -> 0
- net /HDMI0_CK_N: track 0.00 -> 143.9 mm
- net /HDMI0_CK_P: track 0.00 -> 143.8 mm
- net /HDMI0_D0_P: track 0.87 -> 142.2 mm
- net /HDMI0_D0_N: track 0.87 -> 142.1 mm
- net /HDMI0_D1_P: track 0.00 -> 140.4 mm
- net /HDMI0_D1_N: track 0.00 -> 140.2 mm
- net /HDMI0_D2_N: track 0.00 -> 138.4 mm
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Other:
- copper layers 2 -> 4
