File: PiKeyboard/hardware/hardware.kicad_sch (KiCad schematic)
At the start: 7 parts, among them J2 USB_C_Receptacle_PowerOnly_6P, J22 690-019-298-412, U12 RT9742SNGV

Commit message: yes
Connections:
- net HDMI0_CEC: no longer J22.13 (CEC)
- no-connect marks 1 -> 2
Changed lines of the file:
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@@
 		(at 44.45 62.23)
 	)
+	(no_connect
+		(at 44.45 49.53)
+	)
 	(wire
 		(pts
@@
 			(width 0)
 			(type default)
-		)
-	)
-	(wire
-		(pts
-			(xy 27.94 49.53) (xy 44.45 49.53)
-		)
-		(stroke
-			(width 0)
-			(type solid)
 		)
 	)
@@
 		(effects
 			(font
-				(size 1.27 1.27)
-			)
-			(justify left bottom)
-		)
-	)
-	(label "HDMI0_CEC"
-		(at 27.94 49.53 0)
-		(effects
-			(font
