File: PiKeyboard/hardware/matrix.kicad_sch (KiCad schematic)
At the start: 149 parts, among them SW1 SW_Push, SW10 SW_Push, SW11 SW_Push, SW12 SW_Push, SW13 SW_Push, SW14 SW_Push, SW15 SW_Push, SW16 SW_Push, SW17 SW_Push, SW18 SW_Push, SW19 SW_Push, SW2 SW_Push, SW20 SW_Push, SW21 SW_Push, SW22 SW_Push, SW23 SW_Push, SW24 SW_Push, SW25 SW_Push, SW26 SW_Push, SW27 SW_Push, SW28 SW_Push, SW29 SW_Push, SW3 SW_Push, SW30 SW_Push, SW31 SW_Push, SW32 SW_Push, SW33 SW_Push, SW34 SW_Push, SW35 SW_Push, SW36 SW_Push, SW37 SW_Push, SW38 SW_Push, SW39 SW_Push, SW4 SW_Push, SW40 SW_Push, SW41 SW_Push, SW42 SW_Push, SW43 SW_Push, SW44 SW_Push, SW45 SW_Push, SW46 SW_Push, SW47 SW_Push, SW48 SW_Push, SW49 SW_Push, SW5 SW_Push, SW50 SW_Push, SW51 SW_Push, SW52 SW_Push, SW53 SW_Push, SW54 SW_Push, SW55 SW_Push, SW56 SW_Push, SW57 SW_Push, SW58 SW_Push, SW59 SW_Push, SW6 SW_Push, SW60 SW_Push, SW61 SW_Push, SW62 SW_Push, SW63 SW_Push, SW64 SW_Push, SW65 SW_Push, SW66 SW_Push, SW67 SW_Push, SW68 SW_Push, SW69 SW_Push, SW7 SW_Push, SW70 SW_Push, SW71 SW_Push, SW72 SW_Push, SW73 SW_Push, SW74 SW_Push, SW8 SW_Push, SW9 SW_Push

Commit message: yes
Parts:
- added C2: C_Small, Capacitor_SMD:C_0805_2012Metric_Pad1.18x1.45mm_HandSolder, symbol Device:C_Small
Connections:
- net C10: now also A1.9 (GPIO6), SW51.1, SW64.1, SW71.1, SW9.1; no longer SW50.1, SW63.1, SW8.1
- net C11: now also A1.11 (GPIO8), SW10.1, SW52.1, SW65.1, SW72.1; no longer A1.9 (GPIO6), SW51.1, SW64.1, SW9.1
- net C12: now also A1.14 (GPIO10), SW11.1, SW53.1; no longer A1.7 (GPIO5), SW10.1, SW52.1, SW65.1, SW71.1
- net C13: now also A1.16 (GPIO12), SW12.1, SW73.1; no longer A1.6 (GPIO4), SW11.1, SW53.1, SW72.1
- net C14: now also A1.19 (GPIO14), SW13.1, SW27.1, SW41.1, SW54.1, SW66.1, SW74.1; no longer A1.2 (GPIO1), SW12.1, SW73.1
- net C15: no longer A1.1 (GPIO0), SW13.1, SW27.1, SW41.1, SW54.1, SW66.1, SW74.1
- net C2: now also SW43.1, SW56.1
- net C3: now also SW44.1, SW57.1; no longer SW43.1, SW56.1
- net C4: now also SW45.1, SW58.1; no longer SW44.1, SW57.1
- net C5: now also A1.1 (GPIO0), SW46.1, SW59.1; no longer SW45.1, SW58.1
- net C6: now also A1.2 (GPIO1), SW47.1, SW60.1, SW70.1; no longer SW46.1, SW59.1
- net C7: now also A1.4 (GPIO2), SW48.1, SW6.1, SW61.1; no longer SW47.1, SW60.1, SW70.1
- net C8: now also A1.5 (GPIO3), SW49.1, SW62.1, SW7.1; no longer SW48.1, SW6.1, SW61.1
- net C9: now also A1.6 (GPIO4), SW50.1, SW63.1, SW8.1; no longer SW49.1, SW62.1, SW7.1
- net GND: now also C2.1
- net R1: now also A1.20 (GPIO15); no longer A1.4 (GPIO2)
- net R2: now also A1.17 (GPIO13); no longer A1.5 (GPIO3)
- net R3: now also A1.15 (GPIO11)
- net R4: now also A1.12 (GPIO9)
- net R5: now also A1.10 (GPIO7)
- net R6: now also A1.7 (GPIO5)
- net VBUS: now also C2.2
- net at SW49.2: no longer D49.2 (A)
- net at D50.2 (A), SW50.2: now also D49.2 (A)
Other:
- moved on the sheet: D10, D11, D12, D13, D27, D41, D43, D44, D45, D46, D47, D48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
