File: Server-Anywhere/hardware/hardware.kicad_sch (KiCad schematic)
At the start: 9 parts, among them J1 power, J2 USB_C_Receptacle_USB2.0_16P

Commit message: yes
Parts:
- removed H1, H2, H3, H4: MountingHole, MountingHole:MountingHole_3.2mm_M3, symbol Mechanical:MountingHole
- removed J2: USB_C_Receptacle_USB2.0_16P, Connector_USB:USB_C_Receptacle_GCT_USB4105-xx-A_16P_TopMnt_Horizontal, symbol Connector:USB_C_Receptacle_USB2.0_16P
- removed R1, R2: 5k1, Resistor_SMD:R_0805_2012Metric_Pad1.20x1.40mm_HandSolder, symbol Device:R
- added J2: USB_OTG, Connector_USB:USB_Micro-B_Amphenol_10103594-0001LF_Horizontal, symbol Connector:USB_OTG
- added U1: USBLC6-4SC6, Package_TO_SOT_SMD:SOT-23-6, symbol Power_Protection:USBLC6-4SC6
- J1: value power -> USB_C_Receptacle_PowerOnly_6P
Connections:
- net GND: now also J2.5 (GND), J2.6 (Shield), U1.2 (GND)
- net USB_N: now also U1.6 (I/O4)
- net USB_P: now also U1.4 (I/O3)
- net CC1: now reaches Module1.94 (CC1)
- net CC1: now also J1.B5 (CC2); no longer J1.A5 (CC1)
- net CC2: now reaches Module1.96 (CC2)
- net CC2: now also J1.A5 (CC1); no longer J1.B5 (CC2)
- net +5V renamed VBUS
- net VBUS: now also U1.5 (VBUS)
- new net: J2.2 (D-), U1.1 (I/O1)
- new net: J2.3 (D+), U1.3 (I/O2)
Other:
- title: (none) -> Server Anywhere Prototype
